File: kicad/leditaulu.sch (KiCad schematic (older format))
At the start: 49 parts, among them CON1 12V input, P1 Programming header, P2 I2C addr select, P4 I2C addr select, P5 Interconnect 1, P6 Interconnect 2, SW1 SW_RESET, SW2 SW_FLASH, U1 ESP-12E, U2 TLC59116IPWR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

Commit message: Version 1.0
Parts:
- D1: value Schottky -> Schottky 2A
Other:
- moved on the sheet: F1
Changed lines of the file:
@@
 	1    0    0    -1
 $EndComp
-Text GLabel 725  6850 0    40   Input ~ 0
+Text GLabel 675  6850 0    40   Input ~ 0
 VCC
 Text GLabel 3625 6850 2    39   Output ~ 0
@@
 Connection ~ 4625 1550
 Wire Wire Line
-	3525 1550 4825 1550
+	3525 1550 4625 1550
+Wire Wire Line
+	4625 1550 4825 1550
 Wire Wire Line
 	4625 1350 4625 1550
@@
 	1200 1850 1725 1850
 Wire Wire Line
-	4100 3400 4350 3400
+	4100 3400 4250 3400
+Wire Wire Line
+	4250 3400 4350 3400
 Wire Wire Line
 	4250 3275 4250 3400
@@
 	2400 3400 2175 3400
 Wire Wire Line
-	1375 3500 2400 3500
-Wire Wire Line
-	1375 3600 2400 3600
-Wire Wire Line
-	1375 3700 2400 3700
-Wire Wire Line
-	1375 3800 2400 3800
+	1375 3500 1425 3500
+Wire Wire Line
+	1425 3500 2400 3500
+Wire Wire Line
+	1375 3600 1600 3600
+Wire Wire Line
+	1600 3600 2400 3600
+Wire Wire Line
+	1375 3700 1775 3700
+Wire Wire Line
+	1775 3700 2400 3700
+Wire Wire Line
+	1375 3800 1950 3800
+Wire Wire Line
+	1950 3800 2400 3800
 Wire Wire Line
 	1425 3175 1425 3500
@@
 Connection ~ 1950 3800
 Wire Wire Line
-	3525 1350 4350 1350
-Wire Wire Line
-	3525 1450 4350 1450
+	3525 1350 4025 1350
+Wire Wire Line
+	4025 1350 4350 1350
+Wire Wire Line
+	3525 1450 4225 1450
+Wire Wire Line
+	4225 1450 4350 1450
 Wire Wire Line
 	4225 1275 4225 1450
@@
 	5075 1650 5075 1550
 Wire Wire Line
-	3525 1650 5075 1650
+	3525 1650 4300 1650
+Wire Wire Line
+	4300 1650 5075 1650
 Wire Wire Line
 	4675 3700 4100 3700
@@
 	5750 3900 5750 4750
 Wire Wire Line
-	1225 6850 1950 6850
-Wire Wire Line
-	2750 6850 3625 6850
+	1225 6850 1275 6850
+Wire Wire Line
+	1275 6850 1550 6850
+Wire Wire Line
+	1550 6850 1825 6850
+Wire Wire Line
+	1825 6850 1950 6850
+Wire Wire Line
+	2750 6850 2875 6850
+Wire Wire Line
+	2875 6850 3150 6850
+Wire Wire Line
+	3150 6850 3425 6850
+Wire Wire Line
+	3425 6850 3625 6850
 Wire Wire Line
 	2875 7000 2875 6850
 Connection ~ 2875 6850
 Wire Wire Line
-	1825 6725 1825 7000
+	1825 6725 1825 6850
+Wire Wire Line
+	1825 6850 1825 7000
 Connection ~ 1825 6850
 Wire Wire Line
 	1825 7200 1825 7300
 Wire Wire Line
-	1550 7300 3425 7300
-Wire Wire Line
-	2350 7150 2350 7325
+	1550 7300 1825 7300
+Wire Wire Line
+	1825 7300 2350 7300
+Wire Wire Line
+	2350 7300 2875 7300
+Wire Wire Line
+	2875 7300 3150 7300
+Wire Wire Line
+	3150 7300 3425 7300
+Wire Wire Line
+	2350 7150 2350 7300
+Wire Wire Line
+	2350 7300 2350 7325
 Wire Wire Line
 	2875 7300 2875 7200
@@
 	1550 7300 1550 7200
 Wire Wire Line
-	9475 3425 9725 3425
+	9475 3425 9625 3425
+Wire Wire Line
+	9625 3425 9725 3425
 Wire Wire Line
 	9625 3300 9625 3425
@@
 	7775 3425 7550 3425
 Wire Wire Line
-	6750 3525 7775 3525
-Wire Wire Line
-	6750 3625 7775 3625
-Wire Wire Line
-	6750 3725 7775 3725
-Wire Wire Line
-	6750 3825 7775 3825
+	6750 3525 6800 3525
+Wire Wire Line
+	6800 3525 7775 3525
+Wire Wire Line
+	6750 3625 6975 3625
+Wire Wire Line
+	6975 3625 7775 3625
+Wire Wire Line
+	6750 3725 7150 3725
+Wire Wire Line
+	7150 3725 7775 3725
+Wire Wire Line
+	6750 3825 7325 3825
+Wire Wire Line
+	7325 3825 7775 3825
 Wire Wire Line
 	6800 3200 6800 3525
@@
 	11125 3925 11125 4775
 Wire Wire Line
-	4150 6925 5000 6925
+	4150 6925 4425 6925
+Wire Wire Line
+	4425 6925 5000 6925
 Wire Wire Line
 	4750 7075 5000 7075
 Wire Wire Line
-	4750 6425 4750 7075
+	4750 6425 4750 6500
+Wire Wire Line
+	4750 6500 4750 7075
 Wire Wire Line
 	4425 6600 4425 6500
 Wire Wire Line
-	4150 6500 4750 6500
+	4150 6500 4425 6500
+Wire Wire Line
+	4425 6500 4750 6500
 Connection ~ 4750 6500
 Wire Wire Line
@@
 Connection ~ 4425 6500
 Wire Wire Line
-	4425 6800 4425 7000
+	4425 6800 4425 6925
+Wire Wire Line
+	4425 6925 4425 7000
 Wire Wire Line
 	4150 6800 4150 6925
 Connection ~ 4425 6925
 Wire Wire Line
-	3525 1750 4000 1750
+	3525 1750 3775 1750
+Wire Wire Line
+	3775 1750 4000 1750
 Wire Wire Line
 	3775 1750 3775 2025
@@
 $EndComp
 Wire Wire Line
-	1425 1150 1725 1150
+	1425 1150 1575 1150
+Wire Wire Line
+	1575 1150 1725 1150
 Wire Wire Line
 	1575 1050 1575 1150
@@
 L Fuse_Small F1
 U 1 1 5904F150
-P 825 6850
-F 0 "F1" H 825 6790 50  0000 C CNN
-F 1 "2.5A" H 825 6925 50  0000 C CNN
-F 2 "Resistors_SMD:R_0603_HandSoldering" H 825 6850 50  0001 C CNN
-F 3 "" H 825 6850 50  0000 C CNN
-	1    825  6850
+P 775 6850
+F 0 "F1" H 775 6790 50  0000 C CNN
+F 1 "2.5A" H 775 6925 50  0000 C CNN
+F 2 "Resistors_SMD:R_0603_HandSoldering" H 775 6850 50  0001 C CNN
+F 3 "" H 775 6850 50  0000 C CNN
+	1    775  6850
 	1    0    0    -1
 $EndComp
@@
 P 1125 6850
 F 0 "D1" H 1075 6930 50  0000 L CNN
-F 1 "Schottky" H 950 6775 50  0000 L CNN
+F 1 "Schottky 2A" H 850 6775 50  0000 L CNN
 F 2 "Diodes_SMD:D_SOD-123F" V 1125 6850 50  0001 C CNN
 F 3 "" V 1125 6850 50  0000 C CNN
@@
 	1275 7275 1275 7300
 Wire Wire Line
-	1025 6850 925  6850
+	1025 6850 875  6850
 Text GLabel 1825 6725 1    40   Input ~ 0
 VCC_PROT
